File: FuseBit_Doc/USB/atmega_fusebit_doctor_V2_Custom_7_usb.brd (EAGLE design)
At the start: 100 x 100 mm, 73 parts, among them IC1 7805, IC10 MEGA8/88/168..., IC11 MEGA8-AI, IC12 FT232RL, IC14 TINY2313, IC15 MEGA16, IC16 MEGA128-A, IC17 MEGA8/88/168..., IC2 ATMEGA8-DOC, IC3 MEGA16/32/644...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

Commit message: FT232_update
Parts:
- added C6, C8: 100nF, resistor@1:C0805
Connections:
- removed net 3V3OUT: IC12.17
- new net COM: C6.1, C8.1
- new net N$3: C8.2, IC12.17
- net VUSB: now also C6.2, IC12.19
Routing:
- net VUSB: track 47.2 -> 55.6 mm, vias 2 -> 3
- net N$3: track 0.00 -> 6.70 mm
- net BS1: track 169.4 -> 173.9 mm
- net GND: track 363.0 -> 366.1 mm
- net COM: track 0.00 -> 2.62 mm
